File: SensorBoard/SensorBoard.brd (EAGLE design)
At the start: 136.2 x 101 mm, 74 parts, among them IC1 7805, J1 DCJ0202, X1 gen1, X13 3.3out1, X14 3.3out2, X15 uart1, X16 uart2, X17 uart3, X18 uart4, X2 motordriver1, X4 gen2, X5 gen3, X6 gen4, X7 programmer, X8 motordriver2

Commit message: edited some stuff to make it pretty :]
Parts:
- removed U$1, U$2, U$3, U$4: ANTENNA2SMD, SparkFun-RF:ANTENNA-CHIP2
- added U$5, U$6, U$7, U$8: ANTENNA2SMD3, SparkFun-RF:ANTENNA-CHIP4
Connections:
- removed net N$14: GPS4.3, U$4.FEED
- new net N$3: GPS1.3, U$5.SIG
- net N$10: now also GPS2.3, U$7.SIG; no longer GPS1.3, U$1.FEED
- net N$12: now also GPS3.3, U$6.SIG; no longer GPS2.3, U$2.FEED
- net N$13: now also GPS4.3, U$8.SIG; no longer GPS3.3, U$3.FEED
Routing:
- net GND: track 369.5 -> 435.3 mm
- net GPS1XSTB: track 55.3 -> 60.1 mm
- net N$3: track 0.00 -> 4.10 mm
- net N$14: track 3.72 -> 0.00 mm
- net GPS2XSTB: track 56.6 -> 59.7 mm
- net N$13: track 4.93 -> 7.10 mm
Other:
- board text added: "3.3VREG"
- board text added: "C1"
- board text added: "C10"
- board text added: "C11"
- board text added: "C12"
- board text added: "C13"
- board text added: "C14"
- board text added: "C15"
- board text added: "C16"
- board text added: "C17"
- board text added: "C18"
- board text added: "C19"
- board text added: "C2"
- board text added: "C20"
- board text added: "C21"
- board text added: "C3"
- board text added: "C4"
- board text added: "C5"
- board text added: "C6"
- board text added: "C7"
- board text added: "C8"
- board text added: "C9"
- board text added: "CY8C5868AXI-LP035"
- board text added: "IC1"
- board text added: "J1"
- board text added: "LT1763IS8-3.3"
- board text added: "MAGNETO"
- board text added: "MINIUSB"
- board text added: "PI"
- board text added: "PWR"
- board text added: "PWR1"
- board text added: "PWR2"
- board text added: "PWR3"
- board text added: "PWR4"
- board text added: "PWR5"
- board text added: "PWR6"
- board text added: "Quadcopter SensorBoard V1.0"
- board text added: "R1"
- board text added: "R10"
- board text added: "R11"
- board text added: "R12"
- board text added: "R13"
- board text added: "R14"
- board text added: "R15"
- board text added: "R2"
- board text added: "R3"
- board text added: "R4"
- board text added: "R5"
- board text added: "R6"
- board text added: "R7"
- board text added: "R8"
- board text added: "R9"
- board text added: "RC"
- board text added: "U$5"
- board text added: "U$6"
- board text added: "U$7"
- board text added: "U$8"
- board text added: "USBUART"
- board text added: "X1"
- board text added: "X13"
- board text added: "X14"
- board text added: "X15"
- board text added: "X16"
- board text added: "X17"
- board text added: "X18"
- board text added: "X2"
- board text added: "X4"
- board text added: "X5"
- board text added: "X6"
- board text added: "X7"
- board text added: "X8"
- board text removed: "Quadcopter Sensor Board V1.0"
