File: SensorBoard/SensorBoard.sch (EAGLE design)
At the start: 75 parts, among them IC1 7805, J1 DCJ0202, U1 MPU-6000QFN-24, X1 gen1, X13 3.3out1, X14 3.3out2, X15 uart1, X16 uart2, X17 uart3, X18 uart4, X2 motordriver1, X3 MINI-USB-SCHIELD-32005-201, X4 gen2, X5 gen3, X6 gen4, X7 programmer, X8 motordriver2

Commit message: fished SensorBoard.  It is perrrfect! - jack
Parts:
- removed U$5: HMC5883LSMD, SparkFun-Sensors:HMC5883LSMD
- removed U1: MPU-6000QFN-24, SparkFun-Sensors:MPU-6000QFN-24
- removed X3: MINI-USB-SCHIELD-32005-201, con-cypressindustries:MINI-USB-SCHIELD-32005-201
- added ACC: MPU-6000QFN-24, SparkFun-Sensors:MPU-6000QFN-24
- added MAGNETO: HMC5883LSMD, SparkFun-Sensors:HMC5883LSMD
- added MINIUSB: MINI-USB-SCHIELD-32005-201, con-cypressindustries:MINI-USB-SCHIELD-32005-201
Connections:
- new net +3.3VP1: PI-1.S
- new net +3.3VP2: PI-17.S
- new net +5VP1: PI-2.S
- new net +5VP2: PI-4.S
- new net 1: CY8C5868AXI-LP035.P6_1
- new net 2: CY8C5868AXI-LP035.P6_0
- new net 3: CY8C5868AXI-LP035.P4_2
- new net 37: CY8C5868AXI-LP035.P3_5
- new net 44: CY8C5868AXI-LP035.P12_2
- net +3.3V: now also ACC.CS, ACC.VDD, MAGNETO.S1, MAGNETO.VDD, MAGNETO.VDDIO; no longer PI-1.S, PI-17.S, U$5.S1, U$5.VDD, U$5.VDDIO, U1.CS, U1.VDD
- net +5V: no longer PI-2.S, PI-4.S
- net AUXCL1: now also ACC.AUXCL, MAGNETO.SCL; no longer U$5.SCL, U1.AUXCL
- net AUXDA1: now also ACC.AUXDA, MAGNETO.SDA; no longer U$5.SDA, U1.AUXDA
- net CH1: now also CY8C5868AXI-LP035.P3_6; no longer CY8C5868AXI-LP035.P15_0_MXTLO
- net CH2: now also CY8C5868AXI-LP035.P3_7; no longer CY8C5868AXI-LP035.P15_1_MXTLI
- net CH3: now also CY8C5868AXI-LP035.P12_0_I2C1_SCL; no longer CY8C5868AXI-LP035.P3_0
- net CH4: now also CY8C5868AXI-LP035.P12_1_I2C1_SDA; no longer CY8C5868AXI-LP035.P3_3
- net CH5: now also CY8C5868AXI-LP035.P15_2_KXTLO; no longer CY8C5868AXI-LP035.P3_4
- net CH6: now also CY8C5868AXI-LP035.P15_3_KXTLI; no longer CY8C5868AXI-LP035.P3_5
- net CLKOUT1: now also ACC.CLKOUT; no longer U1.CLKOUT
- net CTS#: now also CY8C5868AXI-LP035.P4_1; no longer CY8C5868AXI-LP035.P15_7_DM
- net D+: now also MINIUSBG$1.3; no longer X3G$1.3
- net D-: now also MINIUSBG$1.2; no longer X3G$1.2
- net FSYNC: now also ACC.FSYNC; no longer U1.FSYNC
- net GEN1: now also CY8C5868AXI-LP035.P12_7; no longer CY8C5868AXI-LP035.P5_4
- net GEN2: now also CY8C5868AXI-LP035.P5_4; no longer CY8C5868AXI-LP035.P5_5
- net GEN3: now also CY8C5868AXI-LP035.P5_5; no longer CY8C5868AXI-LP035.P5_6
- net GEN4: now also CY8C5868AXI-LP035.P5_6; no longer CY8C5868AXI-LP035.P5_7
- net GEN5: now also CY8C5868AXI-LP035.P1_7; no longer CY8C5868AXI-LP035.P12_6
- net GEN6: now also CY8C5868AXI-LP035.P12_6; no longer CY8C5868AXI-LP035.P12_7
- net GND: now also ACC.AD0/SDO, ACC.CLKIN, ACC.GND, MAGNETO.GND@1, MAGNETO.GND@2, MINIUSBG$1.1; no longer U$5.GND@1, U$5.GND@2, U1.AD0/SDO, U1.CLKIN, U1.GND, X3G$1.1
- net GPIO10: now also CY8C5868AXI-LP035.P4_7; no longer CY8C5868AXI-LP035.P4_4
- net GPIO11: now also CY8C5868AXI-LP035.P4_5; no longer CY8C5868AXI-LP035.P4_2
- net GPIO14: now also CY8C5868AXI-LP035.P4_4; no longer CY8C5868AXI-LP035.P2_5
- net GPIO15: now also CY8C5868AXI-LP035.P4_3; no longer CY8C5868AXI-LP035.P2_6
- net GPIO17: now also CY8C5868AXI-LP035.P6_2; no longer CY8C5868AXI-LP035.P4_7
- net GPIO18: no longer CY8C5868AXI-LP035.P2_7
- net GPIO2(0): now also CY8C5868AXI-LP035.P15_5; no longer CY8C5868AXI-LP035.P6_2
- net GPIO22: no longer CY8C5868AXI-LP035.P4_5
- net GPIO23: now also CY8C5868AXI-LP035.P0_7; no longer CY8C5868AXI-LP035.P5_0
- net GPIO24: now also CY8C5868AXI-LP035.P0_6; no longer CY8C5868AXI-LP035.P5_1
- net GPIO25: no longer CY8C5868AXI-LP035.P5_2
- net GPIO27: no longer CY8C5868AXI-LP035.P4_6
- net GPIO3(1): now also CY8C5868AXI-LP035.P15_4; no longer CY8C5868AXI-LP035.P6_1
- net GPIO4: now also CY8C5868AXI-LP035.P6_3; no longer CY8C5868AXI-LP035.P6_0
- net GPIO7: no longer CY8C5868AXI-LP035.P3_7
- net GPIO8: no longer CY8C5868AXI-LP035.P5_3
- net GPIO9: now also CY8C5868AXI-LP035.P4_6; no longer CY8C5868AXI-LP035.P4_3
- net GPS1RXA: now also CY8C5868AXI-LP035.P5_3; no longer CY8C5868AXI-LP035.P6_5
- net GPS1RXB: now also CY8C5868AXI-LP035.P1_2; no longer CY8C5868AXI-LP035.P6_7
- net GPS1TXA: now also CY8C5868AXI-LP035.P5_1; no longer CY8C5868AXI-LP035.P6_4
- net GPS1TXB: now also CY8C5868AXI-LP035.P5_2; no longer CY8C5868AXI-LP035.P6_6
- net GPS1XSTB: now also CY8C5868AXI-LP035.P1_3_TDO_SWV; no longer CY8C5868AXI-LP035.P1_2
- net GPS2RXA: now also CY8C5868AXI-LP035.P2_7; no longer CY8C5868AXI-LP035.P2_3
- net GPS2RXB: now also CY8C5868AXI-LP035.P12_4_I2C0_SCL; no longer CY8C5868AXI-LP035.P2_1
- net GPS2TXA: now also CY8C5868AXI-LP035.P2_5; no longer CY8C5868AXI-LP035.P2_4
- net GPS2TXB: now also CY8C5868AXI-LP035.P2_6; no longer CY8C5868AXI-LP035.P2_2
- net GPS2XSTB: now also CY8C5868AXI-LP035.P12_5_I2C0_SDA; no longer CY8C5868AXI-LP035.P1_3_TDO_SWV
- net GPS3RXA: now also CY8C5868AXI-LP035.P6_6; no longer CY8C5868AXI-LP035.P15_5
- net GPS3RXB: now also CY8C5868AXI-LP035.P6_7; no longer CY8C5868AXI-LP035.P6_3
- net GPS3TXA: now also CY8C5868AXI-LP035.P6_4; no longer CY8C5868AXI-LP035.P2_0
- net GPS3TXB: now also CY8C5868AXI-LP035.P6_5; no longer CY8C5868AXI-LP035.P15_4
- net GPS3XSTB: now also CY8C5868AXI-LP035.P5_0; no longer CY8C5868AXI-LP035.P1_4_TDI
- net GPS4RXA: now also CY8C5868AXI-LP035.P2_2; no longer CY8C5868AXI-LP035.P0_6
- net GPS4RXB: now also CY8C5868AXI-LP035.P2_3; no longer CY8C5868AXI-LP035.P0_4
- net GPS4TXA: now also CY8C5868AXI-LP035.P2_0; no longer CY8C5868AXI-LP035.P0_7
- net GPS4TXB: now also CY8C5868AXI-LP035.P2_1; no longer CY8C5868AXI-LP035.P0_5
- net GPS4XSTB: now also CY8C5868AXI-LP035.P2_4; no longer CY8C5868AXI-LP035.P1_5_NTRST
- net INT1: now also ACC.INT, CY8C5868AXI-LP035.P1_6; no longer U1.INT
- net MDTX1: now also CY8C5868AXI-LP035.P5_7; no longer CY8C5868AXI-LP035.P3_2
- net MDTX2: now also CY8C5868AXI-LP035.P15_6_DP; no longer CY8C5868AXI-LP035.P3_1
- net N$11: now also MAGNETO.SETC; no longer U$5.SETC
- net N$15: now also MAGNETO.SETP; no longer U$5.SETP
- net N$16: now also MAGNETO.C1; no longer U$5.C1
- net N$6: now also MINIUSBG$1.4, MINIUSBG$1.5; no longer X3G$1.4, X3G$1.5
- net N$7: now also ACC.REGOUT; no longer U1.REGOUT
- net N$8: now also ACC.CPOUT; no longer U1.CPOUT
- net PWREN#: now also CY8C5868AXI-LP035.P0_3
- net RTS#: now also CY8C5868AXI-LP035.P0_0; no longer CY8C5868AXI-LP035.P15_6_DP
- net RX1: now also CY8C5868AXI-LP035.P0_5; no longer CY8C5868AXI-LP035.P0_3
- net RX2: now also CY8C5868AXI-LP035.P4_0; no longer CY8C5868AXI-LP035.P0_1
- net RX3: now also CY8C5868AXI-LP035.P3_4; no longer CY8C5868AXI-LP035.P4_1
- net RX4: now also CY8C5868AXI-LP035.P3_2; no longer CY8C5868AXI-LP035.P12_3
- net SCL_ACC: now also ACC.SCL/SCLK, CY8C5868AXI-LP035.P1_5_NTRST; no longer CY8C5868AXI-LP035.P12_4_I2C0_SCL, U1.SCL/SCLK
- net SDA_ACC: now also ACC.SDA/SDI, CY8C5868AXI-LP035.P1_4_TDI; no longer CY8C5868AXI-LP035.P12_5_I2C0_SDA, U1.SDA/SDI
- net STATUS1: now also CY8C5868AXI-LP035.P3_0; no longer CY8C5868AXI-LP035.P15_3_KXTLI
- net STATUS2: now also CY8C5868AXI-LP035.P15_1_MXTLI; no longer CY8C5868AXI-LP035.P15_2_KXTLO
- net STATUS3: now also CY8C5868AXI-LP035.P15_0_MXTLO; no longer CY8C5868AXI-LP035.P12_1_I2C1_SDA
- net STATUS4: now also CY8C5868AXI-LP035.P15_7_DM; no longer CY8C5868AXI-LP035.P12_0_I2C1_SCL
- net TX1: now also CY8C5868AXI-LP035.P0_4; no longer CY8C5868AXI-LP035.P0_2
- net TX2: now also CY8C5868AXI-LP035.P12_3; no longer CY8C5868AXI-LP035.P0_0
- net TX3: now also CY8C5868AXI-LP035.P3_3; no longer CY8C5868AXI-LP035.P4_0
- net TX4: now also CY8C5868AXI-LP035.P3_1; no longer CY8C5868AXI-LP035.P12_2
- net USB_RXD: now also CY8C5868AXI-LP035.P0_2; no longer CY8C5868AXI-LP035.P1_6
- net USB_TXD: now also CY8C5868AXI-LP035.P0_1; no longer CY8C5868AXI-LP035.P1_7
Other:
- moved on the sheet: C14, C15, C16, C17, C18, C19, C20, C21, GPS1, GPS2, GPS3, GPS4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

Commit message: most recent version of the board
Parts:
- removed D1: (no value), zetex:DSOD323
Connections:
- removed net N$3: D1.A, J1.1
- net +12V: now also J1.1; no longer D1.C
Changed lines of the file:
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@@
 <part name="P+1" library="supply1" deviceset="+12V" device=""/>
 <part name="GND1" library="supply1" deviceset="GND" device=""/>
-<part name="D1" library="zetex" deviceset="D" device="SOD323"/>
 <part name="GPS1" library="SparkFun-RF" deviceset="COPERNICUS" device="SMD"/>
 <part name="U$1" library="SparkFun-RF" deviceset="ANTENNA2" device="SMD"/>
@@
 <instance part="P+1" gate="1" x="165.1" y="-45.72"/>
 <instance part="GND1" gate="1" x="152.4" y="-66.04"/>
-<instance part="D1" gate="G$1" x="152.4" y="-53.34"/>
 <instance part="GPS1" gate="G$2" x="-132.08" y="-48.26"/>
 <instance part="U$1" gate="G$1" x="-185.42" y="-50.8"/>
@@
 <segment>
 <wire x1="165.1" y1="-53.34" x2="165.1" y2="-48.26" width="0.1524" layer="91"/>
-<wire x1="154.94" y1="-53.34" x2="165.1" y2="-53.34" width="0.1524" layer="91"/>
 <pinref part="P+1" gate="1" pin="+12V"/>
-<pinref part="D1" gate="G$1" pin="C"/>
+<pinref part="J1" gate="G$1" pin="1"/>
+<wire x1="144.78" y1="-53.34" x2="165.1" y2="-53.34" width="0.1524" layer="91"/>
 </segment>
 </net>
@@
 </segment>
 </net>
-<net name="N$3" class="0">
-<segment>
-<wire x1="144.78" y1="-53.34" x2="149.86" y2="-53.34" width="0.1524" layer="91"/>
-<pinref part="J1" gate="G$1" pin="1"/>
-<pinref part="D1" gate="G$1" pin="A"/>
-</segment>
-</net>

Commit message: edited some stuff to make it pretty :]
Parts:
- removed U$1, U$2, U$3, U$4: ANTENNA2SMD, SparkFun-RF:ANTENNA2SMD
- added U$5, U$6, U$7, U$8: ANTENNA2SMD3, SparkFun-RF:ANTENNA2SMD3
Connections:
- removed net N$14: GPS4.RFIN, U$4.SIGNAL
- new net N$3: GPS1.RFIN, U$5.SIGNAL
- net N$10: now also GPS2.RFIN, U$7.SIGNAL; no longer GPS1.RFIN, U$1.SIGNAL
- net N$12: now also GPS3.RFIN, U$6.SIGNAL; no longer GPS2.RFIN, U$2.SIGNAL
- net N$13: now also GPS4.RFIN, U$8.SIGNAL; no longer GPS3.RFIN, U$3.SIGNAL
Changed lines of the file:
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@@
 <setting verticaltext="up"/>
 </settings>
-<grid distance="0.1" unitdist="inch" unit="inch" style="lines" multiple="1" display="no" altdistance="0.01" altunitdist="inch" altunit="inch"/>
+<grid distance="0.1" unitdist="inch" unit="inch" style="lines" multiple="1" display="yes" altdistance="0.01" altunitdist="inch" altunit="inch"/>
 <layers>
 <layer number="1" name="Top" color="4" fill="1" visible="no" active="no"/>
@@
 <part name="GND1" library="supply1" deviceset="GND" device=""/>
 <part name="GPS1" library="SparkFun-RF" deviceset="COPERNICUS" device="SMD"/>
-<part name="U$1" library="SparkFun-RF" deviceset="ANTENNA2" device="SMD"/>
 <part name="GPS2" library="SparkFun-RF" deviceset="COPERNICUS" device="SMD"/>
-<part name="U$2" library="SparkFun-RF" deviceset="ANTENNA2" device="SMD"/>
 <part name="GPS3" library="SparkFun-RF" deviceset="COPERNICUS" device="SMD"/>
-<part name="U$3" library="SparkFun-RF" deviceset="ANTENNA2" device="SMD"/>
 <part name="GPS4" library="SparkFun-RF" deviceset="COPERNICUS" device="SMD"/>
-<part name="U$4" library="SparkFun-RF" deviceset="ANTENNA2" device="SMD"/>
 <part name="X7" library="con-molex" deviceset="KK-156-5" device="" value="programmer"/>
 <part name="PWR" library="led" deviceset="LED" device="" value="GREEN"/>
@@
 <part name="R15" library="resistor" deviceset="R-US_" device="0204/5" value="4k"/>
 <part name="RC" library="RCRECIEVER" deviceset="6-CHANNEL" device=""/>
+<part name="U$5" library="SparkFun-RF" deviceset="ANTENNA2" device="SMD3"/>
+<part name="U$6" library="SparkFun-RF" deviceset="ANTENNA2" device="SMD3"/>
+<part name="U$7" library="SparkFun-RF" deviceset="ANTENNA2" device="SMD3"/>
+<part name="U$8" library="SparkFun-RF" deviceset="ANTENNA2" device="SMD3"/>
 </parts>
 <sheets>
@@
 <instance part="GND1" gate="1" x="152.4" y="-66.04"/>
 <instance part="GPS1" gate="G$2" x="-132.08" y="-48.26"/>
-<instance part="U$1" gate="G$1" x="-185.42" y="-50.8"/>
 <instance part="GPS2" gate="G$2" x="-132.08" y="-109.22"/>
-<instance part="U$2" gate="G$1" x="-185.42" y="-111.76"/>
 <instance part="GPS3" gate="G$2" x="-10.16" y="-48.26"/>
-<instance part="U$3" gate="G$1" x="-63.5" y="-50.8"/>
 <instance part="GPS4" gate="G$2" x="-10.16" y="-109.22"/>
-<instance part="U$4" gate="G$1" x="-63.5" y="-111.76"/>
 <instance part="X7" gate="-1" x="-121.92" y="73.66" rot="R180"/>
 <instance part="X7" gate="-2" x="-121.92" y="76.2" rot="R180"/>
@@
 <instance part="R15" gate="G$1" x="284.48" y="121.92" rot="R90"/>
 <instance part="RC" gate="G$1" x="-119.38" y="116.84" rot="MR0"/>
+<instance part="U$5" gate="G$1" x="-190.5" y="-50.8"/>
+<instance part="U$6" gate="G$1" x="-53.34" y="-50.8"/>
+<instance part="U$7" gate="G$1" x="-190.5" y="-111.76"/>
+<instance part="U$8" gate="G$1" x="-53.34" y="-111.76"/>
 </instances>
 <busses>
@@
 </segment>
 </net>
-<net name="N$10" class="0">
-<segment>
-<pinref part="GPS1" gate="G$2" pin="RFIN"/>
-<wire x1="-137.16" y1="-55.88" x2="-185.42" y2="-55.88" width="0.1524" layer="91"/>
-<pinref part="U$1" gate="G$1" pin="SIGNAL"/>
-</segment>
-</net>
 <net name="GPS1TXA" class="0">
 <segment>
@@
 </segment>
 </net>
-<net name="N$12" class="0">
-<segment>
-<pinref part="GPS2" gate="G$2" pin="RFIN"/>
-<wire x1="-137.16" y1="-116.84" x2="-185.42" y2="-116.84" width="0.1524" layer="91"/>
-<pinref part="U$2" gate="G$1" pin="SIGNAL"/>
-</segment>
-</net>
 <net name="GPS2TXA" class="0">
 <segment>
@@
 </segment>
 </net>
-<net name="N$13" class="0">
-<segment>
-<pinref part="GPS3" gate="G$2" pin="RFIN"/>
-<wire x1="-15.24" y1="-55.88" x2="-63.5" y2="-55.88" width="0.1524" layer="91"/>
-<pinref part="U$3" gate="G$1" pin="SIGNAL"/>
-</segment>
-</net>
 <net name="GPS3TXA" class="0">
 <segment>
@@
 <wire x1="271.78" y1="-73.66" x2="269.24" y2="-73.66" width="0.1524" layer="91"/>
 <label x="256.54" y="-73.66" size="1.778" layer="95"/>
-</segment>
-</net>
-<net name="N$14" class="0">
-<segment>
-<pinref part="GPS4" gate="G$2" pin="RFIN"/>
-<wire x1="-15.24" y1="-116.84" x2="-63.5" y2="-116.84" width="0.1524" layer="91"/>
-<pinref part="U$4" gate="G$1" pin="SIGNAL"/>
 </segment>
 </net>
@@
 </segment>
 </net>
+<net name="N$3" class="0">
+<segment>
+<pinref part="U$5" gate="G$1" pin="SIGNAL"/>
+<pinref part="GPS1" gate="G$2" pin="RFIN"/>
+<wire x1="-190.5" y1="-55.88" x2="-137.16" y2="-55.88" width="0.1524" layer="91"/>
+</segment>
+</net>
+<net name="N$10" class="0">
+<segment>
+<pinref part="U$7" gate="G$1" pin="SIGNAL"/>
+<pinref part="GPS2" gate="G$2" pin="RFIN"/>
+<wire x1="-190.5" y1="-116.84" x2="-137.16" y2="-116.84" width="0.1524" layer="91"/>
+</segment>
+</net>
+<net name="N$12" class="0">
+<segment>
+<pinref part="U$6" gate="G$1" pin="SIGNAL"/>
+<pinref part="GPS3" gate="G$2" pin="RFIN"/>
+<wire x1="-53.34" y1="-55.88" x2="-15.24" y2="-55.88" width="0.1524" layer="91"/>
+</segment>
+</net>
+<net name="N$13" class="0">
+<segment>
+<pinref part="U$8" gate="G$1" pin="SIGNAL"/>
+<pinref part="GPS4" gate="G$2" pin="RFIN"/>
+<wire x1="-53.34" y1="-116.84" x2="-15.24" y2="-116.84" width="0.1524" layer="91"/>
+</segment>
+</net>

Commit message: fixed some errors
Parts:
- PWR, PWR1, PWR2, PWR3, PWR4, PWR5, PWR6: device led:LED -> led:LEDCHIP-LED0603
Changed lines of the file:
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@@
 <setting verticaltext="up"/>
 </settings>
-<grid distance="0.1" unitdist="inch" unit="inch" style="lines" multiple="1" display="yes" altdistance="0.01" altunitdist="inch" altunit="inch"/>
+<grid distance="0.1" unitdist="inch" unit="inch" style="lines" multiple="1" display="no" altdistance="0.01" altunitdist="inch" altunit="inch"/>
 <layers>
 <layer number="1" name="Top" color="4" fill="1" visible="no" active="no"/>
@@
 <part name="GPS4" library="SparkFun-RF" deviceset="COPERNICUS" device="SMD"/>
 <part name="X7" library="con-molex" deviceset="KK-156-5" device="" value="programmer"/>
-<part name="PWR" library="led" deviceset="LED" device="" value="GREEN"/>
+<part name="PWR" library="led" deviceset="LED" device="CHIP-LED0603" value="GREEN"/>
 <part name="R3" library="resistor" deviceset="R-US_" device="0204/5" value="4k"/>
 <part name="ACC" library="SparkFun-Sensors" deviceset="MPU-6000" device="QFN-24"/>
@@
 <part name="X17" library="con-molex" deviceset="KK-156-4" device="" value="uart3"/>
 <part name="X18" library="con-molex" deviceset="KK-156-4" device="" value="uart4"/>
-<part name="PWR1" library="led" deviceset="LED" device="" value="GREEN"/>
-<part name="PWR2" library="led" deviceset="LED" device="" value="GREEN"/>
-<part name="PWR3" library="led" deviceset="LED" device="" value="GREEN"/>
-<part name="PWR4" library="led" deviceset="LED" device="" value="GREEN"/>
+<part name="PWR1" library="led" deviceset="LED" device="CHIP-LED0603" value="GREEN"/>
+<part name="PWR2" library="led" deviceset="LED" device="CHIP-LED0603" value="GREEN"/>
+<part name="PWR3" library="led" deviceset="LED" device="CHIP-LED0603" value="GREEN"/>
+<part name="PWR4" library="led" deviceset="LED" device="CHIP-LED0603" value="GREEN"/>
 <part name="R10" library="resistor" deviceset="R-US_" device="0204/5" value="4k"/>
 <part name="R11" library="resistor" deviceset="R-US_" device="0204/5" value="4k"/>
@@
 <part name="X8" library="con-molex" deviceset="KK-156-3" device="" value="motordriver2"/>
 <part name="PI" library="con-molex" deviceset="87758-2616" device=""/>
-<part name="PWR5" library="led" deviceset="LED" device="" value="GREEN"/>
+<part name="PWR5" library="led" deviceset="LED" device="CHIP-LED0603" value="GREEN"/>
 <part name="R14" library="resistor" deviceset="R-US_" device="0204/5" value="4k"/>
-<part name="PWR6" library="led" deviceset="LED" device="" value="RED"/>
+<part name="PWR6" library="led" deviceset="LED" device="CHIP-LED0603" value="RED"/>
 <part name="R15" library="resistor" deviceset="R-US_" device="0204/5" value="4k"/>
 <part name="RC" library="RCRECIEVER" deviceset="6-CHANNEL" device=""/>
